Commit message: make joint move!

File: src/snake_description/urdf/snake.urdf (robot description, URDF)
Before this commit: robot snake_test, 17 links, 16 joints
Links:
- link base_link: geometry 
Joints:
- removed joint endpoint
- added joint base_link_joint: type fixed, parent base_link, child head, origin xyz=0.0 0.0 0.0 rpy=0.0 1.57075 0.0
