Commit message: snake orientation updated  and gazebo start paused

File: src/snake_sim/snake_description/urdf/snake.xacro (robot description, xacro)
@@ -30,4 +30,5 @@
     <!-- Usage : <xacro:gazebo_links prefix="head"/> -->
     <link name="base_link">
+        <origin xyz="0.0 0.0 0.0"/>
         <!-- <visual>
             <origin xyz="0 0 0.0" rpy="0 -1.57075 0"/>
@@ -40,5 +41,5 @@
         <parent link="base_link"/>
         <child link="head"/>
-        <origin xyz="0.0 0.0 0.0" rpy="0.0 1.57075 0.0"/>
+        <origin xyz="0.0 0.0 0.025" rpy="1.57075 0.0 1.57075"/>
     </joint>
     <link name="head">
