Commit message: simple gaitor log enabled, ground sdf added a.s.o

File: src/snake_sim/kiro_sim/urdf/tmp.urdf (robot description, URDF)
Before this commit: robot kiro_v2, 12 links, 11 joints
Links:
- removed link 10_link
- removed link 11_link
- removed link 12_tail
- removed link 1_head
- removed link 2_link
- removed link 3_link
- removed link 4_link
- removed link 5_link
- removed link 6_link
- removed link 7_link
- removed link 8_link
- removed link 9_link
- added link kiro_v2__10_link, mass 0.192; collision box size=0.005 0.020 0.071; collision cylinder length=.071 radius=.029
- added link kiro_v2__11_link, mass 0.192; collision box size=0.005 0.020 0.071; collision cylinder length=.071 radius=.029
- added link kiro_v2__12_tail, mass 0.192; collision box size=0.005 0.020 0.071; collision cylinder length=.071 radius=.029
- added link kiro_v2__1_head, mass 0.192; collision box size=0.005 0.020 0.092; collision cylinder length=.092 radius=.029
- added link kiro_v2__2_link, mass 0.192; collision box size=0.005 0.020 0.071; collision cylinder length=.071 radius=.029
- added link kiro_v2__3_link, mass 0.192; collision box size=0.005 0.020 0.071; collision cylinder length=.071 radius=.029
- added link kiro_v2__4_link, mass 0.192; collision box size=0.005 0.020 0.071; collision cylinder length=.071 radius=.029
- added link kiro_v2__5_link, mass 0.192; collision box size=0.005 0.020 0.071; collision cylinder length=.071 radius=.029
- added link kiro_v2__6_link, mass 0.192; collision box size=0.005 0.020 0.071; collision cylinder length=.071 radius=.029
- added link kiro_v2__7_link, mass 0.192; collision box size=0.005 0.020 0.071; collision cylinder length=.071 radius=.029
- added link kiro_v2__8_link, mass 0.192; collision box size=0.005 0.020 0.071; collision cylinder length=.071 radius=.029
- added link kiro_v2__9_link, mass 0.192; collision box size=0.005 0.020 0.071; collision cylinder length=.071 radius=.029
Joints:
- removed joint 10_joint
- removed joint 11_joint
- removed joint 1_joint
- removed joint 2_joint
- removed joint 3_joint
- removed joint 4_joint
- removed joint 5_joint
- removed joint 6_joint
- removed joint 7_joint
- removed joint 8_joint
- removed joint 9_joint
- added joint kiro_v2__10_joint: type revolute, parent kiro_v2__10_link, child kiro_v2__11_link, origin xyz=0       0      -0.07099 rpy=0  0  0, axis -1  0  0, limit lower=-1.57079632679 upper=1.57079632679 effort=1.70775 velocity=4.2
- added joint kiro_v2__11_joint: type revolute, parent kiro_v2__11_link, child kiro_v2__12_tail, origin xyz=0       0      -0.07099 rpy=0  0  0, axis 0  1  0, limit lower=-1.57079632679 upper=1.57079632679 effort=1.70775 velocity=4.2
- added joint kiro_v2__1_joint: type revolute, parent kiro_v2__1_head, child kiro_v2__2_link, origin xyz=-0.03549  0       0.029 rpy=0       1.57079  0, axis 0  1  0, limit lower=-1.57079632679 upper=1.57079632679 effort=1.70775 velocity=4.2
- added joint kiro_v2__2_joint: type revolute, parent kiro_v2__2_link, child kiro_v2__3_link, origin xyz=0       0      -0.07099 rpy=0  0  0, axis -1  0  0, limit lower=-1.57079632679 upper=1.57079632679 effort=1.70775 velocity=4.2
- added joint kiro_v2__3_joint: type revolute, parent kiro_v2__3_link, child kiro_v2__4_link, origin xyz=0       0      -0.07099 rpy=0  0  0, axis 0  1  0, limit lower=-1.57079632679 upper=1.57079632679 effort=1.70775 velocity=4.2
- added joint kiro_v2__4_joint: type revolute, parent kiro_v2__4_link, child kiro_v2__5_link, origin xyz=0       0      -0.07099 rpy=0  0  0, axis -1  0  0, limit lower=-1.57079632679 upper=1.57079632679 effort=1.70775 velocity=4.2
- added joint kiro_v2__5_joint: type revolute, parent kiro_v2__5_link, child kiro_v2__6_link, origin xyz=0       0      -0.07099 rpy=0  0  0, axis 0  1  0, limit lower=-1.57079632679 upper=1.57079632679 effort=1.70775 velocity=4.2
- added joint kiro_v2__6_joint: type revolute, parent kiro_v2__6_link, child kiro_v2__7_link, origin xyz=0       0      -0.07099 rpy=0  0  0, axis -1  0  0, limit lower=-1.57079632679 upper=1.57079632679 effort=1.70775 velocity=4.2
- added joint kiro_v2__7_joint: type revolute, parent kiro_v2__7_link, child kiro_v2__8_link, origin xyz=0       0      -0.07099 rpy=0  0  0, axis 0  1  0, limit lower=-1.57079632679 upper=1.57079632679 effort=1.70775 velocity=4.2
- added joint kiro_v2__8_joint: type revolute, parent kiro_v2__8_link, child kiro_v2__9_link, origin xyz=0       0      -0.07099 rpy=0  0  0, axis -1  0  0, limit lower=-1.57079632679 upper=1.57079632679 effort=1.70775 velocity=4.2
- added joint kiro_v2__9_joint: type revolute, parent kiro_v2__9_link, child kiro_v2__10_link, origin xyz=0       0      -0.07099 rpy=0  0  0, axis 0  1  0, limit lower=-1.57079632679 upper=1.57079632679 effort=1.70775 velocity=4.2
